File: tool-display-pcb/Tool-Display-PCB.kicad_sch (KiCad schematic)
At the start: 4 parts, among them J1 4" TFT SPI DISPLAY, J2 ESP32 30-Pin

Commit message: PCB updates, narrower, additional USB option
Parts:
- added J4: Conn_01x05_Pin, Connector_PinHeader_2.54mm:Alex-5pin-microUSB, symbol Connector:Conn_01x05_Pin
Connections:
- net at C1.2, C2.2, J1.LED (Pin_8)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: now also J4.VIN (Pin_5)
- new net: J2.GND (Pin_29), J4.GND (Pin_1)
Changed lines of the file:
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@@
+	)
+	(junction
+		(at 148.59 93.98)
+		(diameter 0)
+		(color 0 0 0 0)
 	)
 	(junction
@@
 	(wire
 		(pts
+			(xy 201.93 93.98) (xy 193.04 93.98)
+		)
+		(stroke
+			(width 0)
+			(type default)
+		)
+	)
+	(wire
+		(pts
 			(xy 138.43 83.82) (xy 154.94 83.82)
 		)
@@
 	(wire
 		(pts
-			(xy 154.94 93.98) (xy 144.78 93.98)
+			(xy 193.04 93.98) (xy 193.04 113.03)
+		)
+		(stroke
+			(width 0)
+			(type default)
+		)
+	)
+	(wire
+		(pts
+			(xy 154.94 93.98) (xy 148.59 93.98)
 		)
 		(stroke
@@
 	(wire
 		(pts
+			(xy 201.93 83.82) (xy 189.23 83.82)
+		)
+		(stroke
+			(width 0)
+			(type default)
+		)
+	)
+	(wire
+		(pts
+			(xy 193.04 113.03) (xy 148.59 113.03)
+		)
+		(stroke
+			(width 0)
+			(type default)
+		)
+	)
+	(wire
+		(pts
 			(xy 133.35 78.74) (xy 133.35 76.2)
 		)
@@
 	(wire
 		(pts
+			(xy 148.59 113.03) (xy 148.59 93.98)
+		)
+		(stroke
+			(width 0)
+			(type default)
+		)
+	)
+	(wire
+		(pts
 			(xy 115.57 76.2) (xy 115.57 93.98)
 		)
@@
 	(wire
 		(pts
+			(xy 189.23 83.82) (xy 189.23 91.44)
+		)
+		(stroke
+			(width 0)
+			(type default)
+		)
+	)
+	(wire
+		(pts
 			(xy 124.46 71.12) (xy 133.35 71.12)
 		)
@@
 	(wire
 		(pts
+			(xy 148.59 93.98) (xy 144.78 93.98)
+		)
+		(stroke
+			(width 0)
+			(type default)
+		)
+	)
+	(wire
+		(pts
 			(xy 124.46 68.58) (xy 135.89 68.58)
 		)
@@
 		(pts
 			(xy 116.84 66.04) (xy 124.46 66.04)
+		)
+		(stroke
+			(width 0)
+			(type default)
+		)
+	)
+	(wire
+		(pts
+			(xy 189.23 91.44) (xy 179.07 91.44)
 		)
 		(stroke
@@
 					(unit 1)
 				)
+			)
+		)
+	)
+	(symbol
+		(lib_id "Connector:Conn_01x05_Pin")
+		(at 196.85 88.9 0)
+		(unit 1)
+		(exclude_from_sim no)
+		(in_bom yes)
+		(on_board yes)
+		(dnp no)
+		(fields_autoplaced yes)
+		(property "Reference" "J4"
+			(at 197.485 78.74 0)
+			(effects
+				(font
+					(size 1.27 1.27)
+				)
+			)
+		)
+		(property "Value" "Conn_01x05_Pin"
+			(at 197.485 81.28 0)
+			(effects
+				(font
+					(size 1.27 1.27)
+				)
+			)
+		)
+		(property "Footprint" "Connector_PinHeader_2.54mm:Alex-5pin-microUSB"
+			(at 196.85 88.9 0)
+			(effects
+				(font
+					(size 1.27 1.27)
+				)
+				(hide yes)
+			)
+		)
+		(property "Datasheet" "~"
+			(at 196.85 88.9 0)
+			(effects
+				(font
+					(size 1.27 1.27)
+				)
+				(hide yes)
+			)
+		)
+		(property "Description" "Generic connector, single row, 01x05, script generated"
+			(at 196.85 88.9 0)
+			(effects
+				(font
+					(size 1.27 1.27)
+				)
+				(hide yes)
+			)
+		)
+		(pin "VIN"
+		)
+		(pin "D+"
+		)
+		(pin "IO"
+		)
+		(pin "GND"
+		)
+		(pin "D-"
+		)
+		(instances
+			(project ""
+				(path "/51aae960-39ca-40c7-bea5-57d9ea889191"
+					(reference "J4")
+					(unit 1)
+				)
